Commit message: Append .gitignore
Append model files

File: mir200_robot_description/urdf/robot.urdf.xacro (robot description, xacro)
@@ -2,4 +2,6 @@
 <robot name="mir200_robot" xmlns:xacro="http://www.ros.org/wiki/xacro">
     <xacro:property name="wheel_diameter" value="0.125"/>
+    <xacro:property name="wheel_seperation" value="0.438"/>
+    <xacro:property name="caster_wheel_seperation" value="0.410"/>
     <link name="base_footprint"/>
     <link name="base_link">
@@ -30,5 +32,5 @@
         <link name="${prefix}_wheel">
             <visual>
-                <origin xyz="0 0 0" rpy="0 0 0"/>
+                <origin xyz="0 0 0" rpy="0 0 ${direction*pi/2}"/>
                 <geometry>
                     <mesh filename="package://mir200_robot_description/meshes/mir200_wheel.dae" scale="1 1 1"/>
@@ -36,5 +38,5 @@
             </visual>
             <collision>
-                <origin xyz="0 0 0" rpy="0 0 0"/>
+                <origin xyz="0 0 0" rpy="0 0 ${direction*pi/2}"/>
                 <geometry>
                     <mesh filename="package://mir200_robot_description/meshes/mir200_wheel.dae" scale="1 1 1"/>
@@ -50,8 +52,119 @@
             <parent link="base_link"/>
             <child link="${prefix}_wheel"/>
-            <origin xyz="0 0 0" rpy="0 0 0"/>
-            <axis="0 1 0"/>
+            <origin xyz="0 ${direction*wheel_seperation/2} 0" rpy="0 0 0"/>
+            <axis xyz="0 1 0"/>
+        </joint>
+    </xacro:macro>
+    <xacro:macro name="insert_front_caster_wheel" params="prefix direction">
+        <link name="${prefix}_front_caster_wheel">
+            <visual>
+                <origin xyz="0 0 0" rpy="0 0 0"/>
+                <geometry>
+                    <mesh filename="package://mir200_robot_description/meshes/mir200_front_caster_wheel.dae" scale="1 1 1"/>
+                </geometry>
+            </visual>
+            <collision>
+                <origin xyz="0 0 0" rpy="0 0 0"/>
+                <geometry>
+                    <mesh filename="package://mir200_robot_description/meshes/mir200_front_caster_wheel.dae" scale="1 1 1"/>
+                </geometry>
+            </collision>
+            <inertial>
+                <origin xyz="0 0 0" rpy="0 0 0"/>
+                <mass value="0.5"/>
+                <inertia ixx="0.0002" ixy="0.0" ixz="0.0" iyy="0.0002" iyz="0.0" izz="0.0003"/>
+            </inertial>
+        </link>
+        <joint name="${prefix}_front_caster_wheel_joint" type="fixed">
+            <parent link="base_link"/>
+            <child link="${prefix}_front_caster_wheel"/>
+            <origin xyz="0.3 ${direction*caster_wheel_seperation/2} 0" rpy="0 0 0"/>
+        </joint>
+    </xacro:macro>
+    <xacro:macro name="insert_rear_caster_wheel" params="prefix direction">
+        <link name="${prefix}_rear_caster_wheel">
+            <visual>
+                <origin xyz="0 0 0" rpy="0 0 0"/>
+                <geometry>
+                    <mesh filename="package://mir200_robot_description/meshes/mir200_rear_caster_wheel.dae" scale="1 1 1"/>
+                </geometry>
+            </visual>
+            <collision>
+                <origin xyz="0 0 0" rpy="0 0 0"/>
+                <geometry>
+                    <mesh filename="package://mir200_robot_description/meshes/mir200_rear_caster_wheel.dae" scale="1 1 1"/>
+                </geometry>
+            </collision>
+            <inertial>
+                <origin xyz="0 0 0" rpy="0 0 0"/>
+                <mass value="0.5"/>
+                <inertia ixx="0.0002" ixy="0.0" ixz="0.0" iyy="0.0002" iyz="0.0" izz="0.0003"/>
+            </inertial>
+        </link>
+        <joint name="${prefix}_rear_caster_wheel_joint" type="fixed">
+            <parent link="base_link"/>
+            <child link="${prefix}_rear_caster_wheel"/>
+            <origin xyz="-0.3 ${direction*caster_wheel_seperation/2} 0" rpy="0 0 0"/>
         </joint>
     </xacro:macro>
     <xacro:insert_wheel prefix="l" direction="1"/>
+    <xacro:insert_wheel prefix="r" direction="-1"/>
+    <xacro:insert_front_caster_wheel prefix="l" direction="1"/>
+    <xacro:insert_front_caster_wheel prefix="r" direction="-1"/>
+    <xacro:insert_rear_caster_wheel prefix="l" direction="1"/>
+    <xacro:insert_rear_caster_wheel prefix="r" direction="-1"/>
+    <link name="front_lidar">
+        <visual>
+            <origin xyz="0 0 0.012" rpy="0 0 0"/>
+            <geometry>
+                <cylinder radius="0.05" length="0.1"/>
+            </geometry>
+            <material name="dark_gray">
+                <color rgba="0.3 0.3 0.3"/>
+            </material>
+        </visual>
+        <collision>
+            <origin xyz="0 0 0" rpy="0 0 0"/>
+            <geometry>
+                <cylinder radius="0.02" length="0.02"/>
+            </geometry>
+        </collision>
+        <inertial>
+            <origin xyz="0 0 0" rpy="0 0 0"/>
+            <mass value="0.5"/>
+            <inertia ixx="0.0002" ixy="0.0" ixz="0.0" iyy="0.0002" iyz="0.0" izz="0.0003"/>
+        </inertial>
+    </link>
+    <joint name="front_lidar_fixed" type="fixed">
+        <parent link="base_link"/>
+        <child link="front_lidar"/>
+        <origin xyz="0.426 0.235 0.13" rpy="0 0 0"/>
+    </joint>
+    <link name="rear_lidar">
+        <visual>
+            <origin xyz="0 0 0.012" rpy="0 0 0"/>
+            <geometry>
+                <cylinder radius="0.05" length="0.1"/>
+            </geometry>
+            <material name="dark_gray">
+                <color rgba="0.3 0.3 0.3"/>
+            </material>
+        </visual>
+        <collision>
+            <origin xyz="0 0 0" rpy="0 0 0"/>
+            <geometry>
+                <cylinder radius="0.02" length="0.02"/>
+            </geometry>
+        </collision>
+        <inertial>
+            <origin xyz="0 0 0" rpy="0 0 0"/>
+            <mass value="0.5"/>
+            <inertia ixx="0.0002" ixy="0.0" ixz="0.0" iyy="0.0002" iyz="0.0" izz="0.0003"/>
+        </inertial>
+    </link>
+    <joint name="rear_lidar_fixed" type="fixed">
+        <parent link="base_link"/>
+        <child link="rear_lidar"/>
+        <origin xyz="-0.360 -0.235 0.13" rpy="0 0 ${pi}"/>
+    </joint>
 </robot>

Commit message: Add gazebo package for simulation

File: mir200_robot_description/urdf/robot.urdf.xacro (robot description, xacro)
@@ -1,7 +1,16 @@
 <?xml version="1.0" ?>
 <robot name="mir200_robot" xmlns:xacro="http://www.ros.org/wiki/xacro">
+    <!-- include other files -->
+    <xacro:include filename="$(find mir200_robot_description)/urdf/gazebo.urdf.xacro" />
+    <xacro:include filename="$(find mir200_robot_description)/urdf/inertial_macro.xacro" />
+    <!-- robot specifications -->
     <xacro:property name="wheel_diameter" value="0.125"/>
     <xacro:property name="wheel_seperation" value="0.438"/>
     <xacro:property name="caster_wheel_seperation" value="0.410"/>
+    <xacro:property name="robot_weight" value="65.0"/>
+    <xacro:property name="robot_length" value="0.890"/>
+    <xacro:property name="robot_width" value="0.580"/>
+    <xacro:property name="robot_height" value="0.305"/>
+    <!-- URDF -->
     <link name="base_footprint"/>
     <link name="base_link">
@@ -19,7 +28,7 @@
         </collision>
         <inertial>
-            <mass value="0.01"/>
-            <origin xyz="0 0 0" rpy="0 0 0"/>
-            <inertia ixx="0.0001" ixy="0.0" ixz="0.0" iyy="0.0001" iyz="0.0" izz="0.0001"/>
+            <mass value="${robot_weight}"/>
+            <origin xyz="0 0 0.150" rpy="0 0 0"/>
+            <xacro:box_inertia m="${robot_weight}" x="${robot_length}" y="${robot_width}" z="${robot_height}"/>
         </inertial>
     </link>
@@ -44,7 +53,7 @@
             </collision>
             <inertial>
-                <origin xyz="0 0 0" rpy="0 0 0"/>
-                <mass value="0.5"/>
-                <inertia ixx="0.0002" ixy="0.0" ixz="0.0" iyy="0.0002" iyz="0.0" izz="0.0003"/>
+                <origin xyz="0 0 0" rpy="${pi/2} 0 0"/>
+                <mass value="1.0"/>
+                <xacro:cylinder_inertia m="1.0" r="0.0625" h="0.0345"/>
             </inertial>
         </link>
@@ -72,6 +81,6 @@
             <inertial>
                 <origin xyz="0 0 0" rpy="0 0 0"/>
-                <mass value="0.5"/>
-                <inertia ixx="0.0002" ixy="0.0" ixz="0.0" iyy="0.0002" iyz="0.0" izz="0.0003"/>
+                <mass value="1.0"/>
+                <xacro:cylinder_inertia m="1.0" r="0.0625" h="0.032"/>
             </inertial>
         </link>
@@ -79,5 +88,5 @@
             <parent link="base_link"/>
             <child link="${prefix}_front_caster_wheel"/>
-            <origin xyz="0.3 ${direction*caster_wheel_seperation/2} 0" rpy="0 0 0"/>
+            <origin xyz="0.3 ${direction*caster_wheel_seperation/2} 0.001" rpy="0 0 0"/>
         </joint>
     </xacro:macro>
@@ -98,6 +107,6 @@
             <inertial>
                 <origin xyz="0 0 0" rpy="0 0 0"/>
-                <mass value="0.5"/>
-                <inertia ixx="0.0002" ixy="0.0" ixz="0.0" iyy="0.0002" iyz="0.0" izz="0.0003"/>
+                <mass value="1.0"/>
+                <xacro:cylinder_inertia m="1.0" r="0.0625" h="0.032"/>
             </inertial>
         </link>
@@ -105,5 +114,5 @@
             <parent link="base_link"/>
             <child link="${prefix}_rear_caster_wheel"/>
-            <origin xyz="-0.3 ${direction*caster_wheel_seperation/2} 0" rpy="0 0 0"/>
+            <origin xyz="-0.3 ${direction*caster_wheel_seperation/2} 0.001" rpy="0 0 0"/>
         </joint>
     </xacro:macro>
@@ -125,7 +134,7 @@
         </visual>
         <collision>
-            <origin xyz="0 0 0" rpy="0 0 0"/>
+            <origin xyz="0 0 0.012" rpy="0 0 0"/>
             <geometry>
-                <cylinder radius="0.02" length="0.02"/>
+                <cylinder radius="0.05" length="0.1"/>
             </geometry>
         </collision>
@@ -133,5 +142,5 @@
             <origin xyz="0 0 0" rpy="0 0 0"/>
             <mass value="0.5"/>
-            <inertia ixx="0.0002" ixy="0.0" ixz="0.0" iyy="0.0002" iyz="0.0" izz="0.0003"/>
+            <xacro:cylinder_inertia m="0.5" r="0.005" h="0.1"/>
         </inertial>
     </link>
@@ -152,7 +161,7 @@
         </visual>
         <collision>
-            <origin xyz="0 0 0" rpy="0 0 0"/>
+            <origin xyz="0 0 0.012" rpy="0 0 0"/>
             <geometry>
-                <cylinder radius="0.02" length="0.02"/>
+                <cylinder radius="0.05" length="0.1"/>
             </geometry>
         </collision>
@@ -160,5 +169,5 @@
             <origin xyz="0 0 0" rpy="0 0 0"/>
             <mass value="0.5"/>
-            <inertia ixx="0.0002" ixy="0.0" ixz="0.0" iyy="0.0002" iyz="0.0" izz="0.0003"/>
+            <xacro:cylinder_inertia m="0.5" r="0.005" h="0.1"/>
         </inertial>
     </link>
@@ -167,4 +176,4 @@
         <child link="rear_lidar"/>
         <origin xyz="-0.360 -0.235 0.13" rpy="0 0 ${pi}"/>
-    </joint>
+    </joint> -->
 </robot>
