Commit message: Bug fixed

File: mir200_w_ur5e_robot_description/urdf/gazebo.urdf.xacro (robot description, xacro)
@@ -22,4 +22,16 @@
         <mu1>0.0</mu1>
         <mu2>0.0</mu2>
+    </gazebo>
+    <gazebo reference="l_wheel">
+        <mu1>100.0</mu1>
+        <mu2>100.0</mu2>
+        <kp value="10000.0" />
+        <kd value="1.0" />
+    </gazebo>
+    <gazebo reference="r_wheel">
+        <mu1>100.0</mu1>
+        <mu2>100.0</mu2>
+        <kp value="10000.0" />
+        <kd value="1.0" />
     </gazebo>
     <gazebo>

File: mir200_w_ur5e_robot_description/urdf/robot.urdf.xacro (robot description, xacro)
@@ -1,4 +1,11 @@
 <?xml version="1.0" ?>
 <robot name="mir200_w_ur5e_robot" xmlns:xacro="http://www.ros.org/wiki/xacro">
+    <!-- UR Related -->
+    <xacro:arg name="transmission_hw_interface" default="hardware_interface/PositionJointInterface"/>
+    <xacro:include filename="$(find ur_description)/urdf/common.gazebo.xacro" />
+    <xacro:include filename="$(find ur_e_description)/urdf/ur5e.urdf.xacro" />
+    <xacro:arg name="kinematics_config" default="$(find ur_e_description)/config/ur5e_default.yaml"/>
+    <!-- Robotiq Gripper -->
+    <xacro:include filename="$(find robotiq_2f_85_gripper_visualization)/urdf/robotiq_arg2f_85_model_macro.xacro" />
     <!-- include other files -->
     <xacro:include filename="$(find mir200_w_ur5e_robot_description)/urdf/gazebo.urdf.xacro" />
@@ -12,5 +19,5 @@
     <xacro:property name="robot_width" value="0.580"/>
     <xacro:property name="robot_height" value="0.305"/>
-    <!-- URDF -->
+    <!-- Mobile Base MIR200 -->
     <link name="base_footprint"/>
     <link name="base_link">
@@ -88,5 +95,5 @@
             <parent link="base_link"/>
             <child link="${prefix}_front_caster_wheel"/>
-            <origin xyz="0.3 ${direction*caster_wheel_seperation/2} 0.001" rpy="0 0 0"/>
+            <origin xyz="0.3 ${direction*caster_wheel_seperation/2} 0.0001" rpy="0 0 0"/>
         </joint>
     </xacro:macro>
@@ -114,5 +121,5 @@
             <parent link="base_link"/>
             <child link="${prefix}_rear_caster_wheel"/>
-            <origin xyz="-0.3 ${direction*caster_wheel_seperation/2} 0.001" rpy="0 0 0"/>
+            <origin xyz="-0.3 ${direction*caster_wheel_seperation/2} 0.0001" rpy="0 0 0"/>
         </joint>
     </xacro:macro>
@@ -123,4 +130,5 @@
     <xacro:insert_rear_caster_wheel prefix="l" direction="1"/>
     <xacro:insert_rear_caster_wheel prefix="r" direction="-1"/>
+    <!-- Front / Rear Lidar -->
     <link name="front_lidar">
         <visual>
@@ -129,6 +137,6 @@
                 <cylinder radius="0.05" length="0.1"/>
             </geometry>
-            <material name="dark_gray">
-                <color rgba="0.3 0.3 0.3"/>
+            <material name="dark_yellow">
+                <color rgba="0.6 0.6 0.3 1.0"/>
             </material>
         </visual>
@@ -156,6 +164,6 @@
                 <cylinder radius="0.05" length="0.1"/>
             </geometry>
-            <material name="dark_gray">
-                <color rgba="0.3 0.3 0.3"/>
+            <material name="dark_yellow">
+                <color rgba="0.6 0.6 0.3 1.0"/>
             </material>
         </visual>
@@ -177,3 +185,50 @@
         <origin xyz="-0.360 -0.235 0.13" rpy="0 0 ${pi}"/>
     </joint>
+    <!-- Mount Box -->
+    <link name="mount_box">
+        <visual>
+            <origin xyz="0 0 0" rpy="0 0 0"/>
+            <geometry>
+                <mesh filename="package://mir200_w_ur5e_robot_description/meshes/mir200_mount_box.dae" scale="1 1 1"/>
+            </geometry>
+        </visual>
+        <collision>
+            <origin xyz="0 0 0" rpy="0 0 0"/>
+            <geometry>
+                <mesh filename="package://mir200_w_ur5e_robot_description/meshes/mir200_mount_box.dae" scale="1 1 1"/>
+            </geometry>
+        </collision>
+        <inertial>
+            <origin xyz="0 0 0" rpy="0 0 0"/>
+            <mass value="10.0"/>
+            <xacro:box_inertia m="10.0" x="0.750" y="0.4" z="0.45"/>
+        </inertial>
+    </link>
+    <joint name="mount_box_fixed" type="fixed">
+        <parent link="base_link"/>
+        <child link="mount_box"/>
+        <origin xyz="0.035 0 0.295" rpy="0 0 0"/>
+    </joint>
+    <!-- UR5e -->
+    <xacro:ur5e_robot prefix="ur5e_" joint_limited="true"
+        shoulder_pan_lower_limit="${-pi}" shoulder_pan_upper_limit="${pi}"
+        shoulder_lift_lower_limit="${-pi}" shoulder_lift_upper_limit="${pi}"
+        elbow_joint_lower_limit="${-pi}" elbow_joint_upper_limit="${pi}"
+        wrist_1_lower_limit="${-pi}" wrist_1_upper_limit="${pi}"
+        wrist_2_lower_limit="${-pi}" wrist_2_upper_limit="${pi}"
+        wrist_3_lower_limit="${-pi}" wrist_3_upper_limit="${pi}"
+        kinematics_file="${load_yaml('$(arg kinematics_config)')}"
+    />
+    <joint name="ur5e_mount_fixed" type="fixed">
+        <parent link="mount_box"/>
+        <child link="ur5e_base_link"/>
+        <origin xyz="-0.2 0 0.45" rpy="0 0 0"/>
+    </joint>
+    <!-- Robotiq Gripper -->
+    <xacro:robotiq_arg2f_85 prefix=""/>
+    <joint name="ur5e_tool0_to_gripper" type="fixed">
+        <parent link="ur5e_tool0"/>
+        <child link="robotiq_arg2f_base_link"/>
+        <origin xyz="0 0 0" rpy="0 0 ${pi/2}"/>
+    </joint>
 </robot>

Commit message: Reduce the faces of meshes
Change the collision of caster wheels from mesh to cylinder

File: mir200_w_ur5e_robot_description/urdf/gazebo.urdf.xacro (robot description, xacro)
@@ -26,12 +26,14 @@
         <mu1>100.0</mu1>
         <mu2>100.0</mu2>
+        <!--
         <kp value="10000.0" />
-        <kd value="1.0" />
+        <kd value="1.0" /> -->
     </gazebo>
     <gazebo reference="r_wheel">
         <mu1>100.0</mu1>
         <mu2>100.0</mu2>
+        <!--
         <kp value="10000.0" />
-        <kd value="1.0" />
+        <kd value="1.0" /> -->
     </gazebo>
     <gazebo>

File: mir200_w_ur5e_robot_description/urdf/robot.urdf.xacro (robot description, xacro)
@@ -54,7 +54,8 @@
             </visual>
             <collision>
-                <origin xyz="0 0 0" rpy="0 0 ${direction*pi/2}"/>
-                <geometry>
-                    <mesh filename="package://mir200_w_ur5e_robot_description/meshes/mir200_wheel.dae" scale="1 1 1"/>
+                <origin xyz="0 0 0" rpy="${pi/2} 0 0"/>
+                <geometry>
+                    <!-- <mesh filename="package://mir200_w_ur5e_robot_description/meshes/mir200_wheel.dae" scale="1 1 1"/> -->
+                    <cylinder radius="0.0625" length="0.0345"/>
                 </geometry>
             </collision>
@@ -68,5 +69,5 @@
             <parent link="base_link"/>
             <child link="${prefix}_wheel"/>
-            <origin xyz="0 ${direction*wheel_seperation/2} 0" rpy="0 0 0"/>
+            <origin xyz="0 ${direction*wheel_seperation/2} 0.0" rpy="0 0 0"/>
             <axis xyz="0 1 0"/>
         </joint>
@@ -81,7 +82,8 @@
             </visual>
             <collision>
-                <origin xyz="0 0 0" rpy="0 0 0"/>
-                <geometry>
-                    <mesh filename="package://mir200_w_ur5e_robot_description/meshes/mir200_front_caster_wheel.dae" scale="1 1 1"/>
+                <origin xyz="0 0 0" rpy="${pi/2} 0 0"/>
+                <geometry>
+                    <!-- <mesh filename="package://mir200_w_ur5e_robot_description/meshes/mir200_front_caster_wheel.dae" scale="1 1 1"/> -->
+                    <cylinder radius="0.0625" length="0.032"/>
                 </geometry>
             </collision>
@@ -95,5 +97,5 @@
             <parent link="base_link"/>
             <child link="${prefix}_front_caster_wheel"/>
-            <origin xyz="0.3 ${direction*caster_wheel_seperation/2} 0.0001" rpy="0 0 0"/>
+            <origin xyz="0.3 ${direction*caster_wheel_seperation/2} 0.001" rpy="0 0 0"/>
         </joint>
     </xacro:macro>
@@ -107,7 +109,8 @@
             </visual>
             <collision>
-                <origin xyz="0 0 0" rpy="0 0 0"/>
-                <geometry>
-                    <mesh filename="package://mir200_w_ur5e_robot_description/meshes/mir200_rear_caster_wheel.dae" scale="1 1 1"/>
+                <origin xyz="0 0 0" rpy="${pi/2} 0 0"/>
+                <geometry>
+                    <!-- <mesh filename="package://mir200_w_ur5e_robot_description/meshes/mir200_rear_caster_wheel.dae" scale="1 1 1"/> -->
+                    <cylinder radius="0.0625" length="0.032"/>
                 </geometry>
             </collision>
@@ -121,5 +124,5 @@
             <parent link="base_link"/>
             <child link="${prefix}_rear_caster_wheel"/>
-            <origin xyz="-0.3 ${direction*caster_wheel_seperation/2} 0.0001" rpy="0 0 0"/>
+            <origin xyz="-0.3 ${direction*caster_wheel_seperation/2} 0.001" rpy="0 0 0"/>
         </joint>
     </xacro:macro>
