Commit message: Change the package names

File: mir200_w_ur5e_robot_description/urdf/robot.urdf.xacro (robot description, xacro)
@@ -1,7 +1,7 @@
 <?xml version="1.0" ?>
-<robot name="mir200_robot" xmlns:xacro="http://www.ros.org/wiki/xacro">
+<robot name="mir200_w_ur5e_robot" xmlns:xacro="http://www.ros.org/wiki/xacro">
     <!-- include other files -->
-    <xacro:include filename="$(find mir200_robot_description)/urdf/gazebo.urdf.xacro" />
-    <xacro:include filename="$(find mir200_robot_description)/urdf/inertial_macro.xacro" />
+    <xacro:include filename="$(find mir200_w_ur5e_robot_description)/urdf/gazebo.urdf.xacro" />
+    <xacro:include filename="$(find mir200_w_ur5e_robot_description)/urdf/inertial_macro.xacro" />
     <!-- robot specifications -->
     <xacro:property name="wheel_diameter" value="0.125"/>
@@ -18,5 +18,5 @@
             <origin xyz="0 0 0" rpy="0 0 0"/>
             <geometry>
-                <mesh filename="package://mir200_robot_description/meshes/mir200_base.dae" scale="1 1 1"/>
+                <mesh filename="package://mir200_w_ur5e_robot_description/meshes/mir200_base.dae" scale="1 1 1"/>
             </geometry>
         </visual>
@@ -24,5 +24,5 @@
             <origin xyz="0 0 0" rpy="0 0 0"/>
             <geometry>
-                <mesh filename="package://mir200_robot_description/meshes/mir200_base.dae" scale="1 1 1"/>
+                <mesh filename="package://mir200_w_ur5e_robot_description/meshes/mir200_base.dae" scale="1 1 1"/>
             </geometry>
         </collision>
@@ -43,5 +43,5 @@
                 <origin xyz="0 0 0" rpy="0 0 ${direction*pi/2}"/>
                 <geometry>
-                    <mesh filename="package://mir200_robot_description/meshes/mir200_wheel.dae" scale="1 1 1"/>
+                    <mesh filename="package://mir200_w_ur5e_robot_description/meshes/mir200_wheel.dae" scale="1 1 1"/>
                 </geometry>
             </visual>
@@ -49,5 +49,5 @@
                 <origin xyz="0 0 0" rpy="0 0 ${direction*pi/2}"/>
                 <geometry>
-                    <mesh filename="package://mir200_robot_description/meshes/mir200_wheel.dae" scale="1 1 1"/>
+                    <mesh filename="package://mir200_w_ur5e_robot_description/meshes/mir200_wheel.dae" scale="1 1 1"/>
                 </geometry>
             </collision>
@@ -70,5 +70,5 @@
                 <origin xyz="0 0 0" rpy="0 0 0"/>
                 <geometry>
-                    <mesh filename="package://mir200_robot_description/meshes/mir200_front_caster_wheel.dae" scale="1 1 1"/>
+                    <mesh filename="package://mir200_w_ur5e_robot_description/meshes/mir200_front_caster_wheel.dae" scale="1 1 1"/>
                 </geometry>
             </visual>
@@ -76,5 +76,5 @@
                 <origin xyz="0 0 0" rpy="0 0 0"/>
                 <geometry>
-                    <mesh filename="package://mir200_robot_description/meshes/mir200_front_caster_wheel.dae" scale="1 1 1"/>
+                    <mesh filename="package://mir200_w_ur5e_robot_description/meshes/mir200_front_caster_wheel.dae" scale="1 1 1"/>
                 </geometry>
             </collision>
@@ -96,5 +96,5 @@
                 <origin xyz="0 0 0" rpy="0 0 0"/>
                 <geometry>
-                    <mesh filename="package://mir200_robot_description/meshes/mir200_rear_caster_wheel.dae" scale="1 1 1"/>
+                    <mesh filename="package://mir200_w_ur5e_robot_description/meshes/mir200_rear_caster_wheel.dae" scale="1 1 1"/>
                 </geometry>
             </visual>
@@ -102,5 +102,5 @@
                 <origin xyz="0 0 0" rpy="0 0 0"/>
                 <geometry>
-                    <mesh filename="package://mir200_robot_description/meshes/mir200_rear_caster_wheel.dae" scale="1 1 1"/>
+                    <mesh filename="package://mir200_w_ur5e_robot_description/meshes/mir200_rear_caster_wheel.dae" scale="1 1 1"/>
                 </geometry>
             </collision>
@@ -176,4 +176,4 @@
         <child link="rear_lidar"/>
         <origin xyz="-0.360 -0.235 0.13" rpy="0 0 ${pi}"/>
-    </joint> -->
+    </joint>
 </robot>

Commit message: Add moveit_client for demo

File: mir200_w_ur5e_robot_description/urdf/robot.urdf.xacro (robot description, xacro)
@@ -232,3 +232,10 @@
         <origin xyz="0 0 0" rpy="0 0 ${pi/2}"/>
     </joint>
+    <!-- EEF for grasp -->
+    <link name="gripper_eef" />
+    <joint name="gipper_eef_fixed" type="fixed">
+        <parent link="robotiq_arg2f_base_link"/>
+        <child link="gripper_eef" />
+        <origin xyz="0 0 0.13" rpy="0 0 0"/>
+    </joint>
 </robot>

Commit message: Change the mass

File: mir200_w_ur5e_robot_description/urdf/robot.urdf.xacro (robot description, xacro)
@@ -15,5 +15,5 @@
     <xacro:property name="wheel_seperation" value="0.438"/>
     <xacro:property name="caster_wheel_seperation" value="0.410"/>
-    <xacro:property name="robot_weight" value="65.0"/>
+    <xacro:property name="robot_weight" value="100.0"/>
     <xacro:property name="robot_length" value="0.890"/>
     <xacro:property name="robot_width" value="0.580"/>
@@ -62,6 +62,6 @@
             <inertial>
                 <origin xyz="0 0 0" rpy="${pi/2} 0 0"/>
-                <mass value="1.0"/>
-                <xacro:cylinder_inertia m="1.0" r="0.0625" h="0.0345"/>
+                <mass value="10.0"/>
+                <xacro:cylinder_inertia m="10.0" r="0.0625" h="0.0345"/>
             </inertial>
         </link>
@@ -90,6 +90,6 @@
             <inertial>
                 <origin xyz="0 0 0" rpy="0 0 0"/>
-                <mass value="1.0"/>
-                <xacro:cylinder_inertia m="1.0" r="0.0625" h="0.032"/>
+                <mass value="10.0"/>
+                <xacro:cylinder_inertia m="10.0" r="0.0625" h="0.032"/>
             </inertial>
         </link>
@@ -117,6 +117,6 @@
             <inertial>
                 <origin xyz="0 0 0" rpy="0 0 0"/>
-                <mass value="1.0"/>
-                <xacro:cylinder_inertia m="1.0" r="0.0625" h="0.032"/>
+                <mass value="10.0"/>
+                <xacro:cylinder_inertia m="10.0" r="0.0625" h="0.032"/>
             </inertial>
         </link>
