Commit message: Adjust parameters

File: mobile_manipulator_robot_description/urdf/bogie_mobile_robot.urdf.xacro (robot description, xacro)
@@ -63,5 +63,6 @@
                     <mass value="5.0"/>
                     <origin xyz="0 ${-dir*0.01} 0" rpy="0 0 0"/>
-                    <xacro:box_inertia m="5.0" x="0.24" y="0.06" z="0.06"/>
+                    <!-- <xacro:box_inertia m="5.0" x="0.24" y="0.06" z="0.06"/> -->
+                    <inertia ixx="1.0" ixy="0" ixz="0" iyy="1.0" iyz="0" izz="1.0" />
                 </inertial>
             </link>
