Commit message: Add rgbd camera for 3d perception

File: mobile_manipulator_robot_description/urdf/gazebo.urdf.xacro (robot description, xacro)
@@ -153,3 +153,39 @@
         </sensor>
     </gazebo>
+    <gazebo reference="camera_link">
+        <sensor type="depth" name="camera">
+            <always_on>true</always_on>
+            <update_rate>30.0</update_rate>
+            <camera>
+                <horizontal_fov>${60.0*pi/180.0}</horizontal_fov>
+                <image>
+                    <format>R8G8B8</format>
+                    <width>640</width>
+                    <height>480</height>
+                </image>
+                <clip>
+                    <near>0.05</near>
+                    <far>8.0</far>
+                </clip>
+            </camera>
+            <plugin name="kinect_camera_controller" filename="libgazebo_ros_openni_kinect.so">
+                <cameraName>camera</cameraName>
+                <alwaysOn>true</alwaysOn>
+                <updateRate>30</updateRate>
+                <imageTopicName>rgb/image_raw</imageTopicName>
+                <depthImageTopicName>depth_registered/image_raw</depthImageTopicName>
+                <pointCloudTopicName>depth_registered/points</pointCloudTopicName>
+                <cameraInfoTopicName>rgb/camera_info</cameraInfoTopicName>
+                <depthImageCameraInfoTopicName>depth_registered/camera_info</depthImageCameraInfoTopicName>
+                <frameName>camera_depth_optical_frame</frameName>
+                <baseline>0.1</baseline>
+                <distortion_k1>0.0</distortion_k1>
+                <distortion_k2>0.0</distortion_k2>
+                <distortion_k3>0.0</distortion_k3>
+                <distortion_t1>0.0</distortion_t1>
+                <distortion_t2>0.0</distortion_t2>
+                <pointCloudCutoff>0.4</pointCloudCutoff>
+            </plugin>
+        </sensor>
+    </gazebo>
 </robot>

File: mobile_manipulator_robot_description/urdf/robot.urdf.xacro (robot description, xacro)
@@ -11,4 +11,6 @@
     <!-- Mobile Robot -->
     <xacro:bogie_mobile_robot/>
+    <!-- D435 -->
+    <xacro:include filename="$(find realsense2_description)/urdf/_d435.urdf.xacro" />
     <!-- Mount Box -->
     <link name="mount_box">
@@ -65,3 +67,6 @@
         <origin xyz="0 0 0.13" rpy="0 0 0"/>
     </joint>
+    <xacro:sensor_d435 parent="mount_box" use_nominal_extrinsics="$(arg use_nominal_extrinsics)">
+        <origin xyz="-0.37 0 0.435" rpy="0 0 ${pi}"/>
+    </xacro:sensor_d435>
 </robot>
